Commit message: Changes to accomodate LOCUS

File: src/multi_jackal/multi_jackal_description/urdf/base_accessories.urdf.xacro (robot description, xacro)
@@ -22,5 +22,5 @@
     <xacro:if value="${lidar_3d_model == 'vlp16'}">
       <xacro:vlp16_mount topic="${topic}" tower="${tower}" prefix="${prefix}" parent_link="${parent}" >
-        <origin xyz="$(optenv JACKAL_LASER_3D_OFFSET 0 0 0)" rpy="$(optenv JACKAL_LASER_3D_RPY 0 0 ${M_PI_Half})" />
+        <origin xyz="$(optenv JACKAL_LASER_3D_OFFSET 0 0 0)" rpy="$(optenv JACKAL_LASER_3D_RPY 0 0 0)" />
       </xacro:vlp16_mount>
     </xacro:if>
