Commit message: Changes to enhance movebase

File: src/multi_jackal/multi_jackal_description/urdf/jackal_with_realsense.urdf.xacro (robot description, xacro)
@@ -38,5 +38,5 @@
       <inertial>
         <origin xyz="0 0 0" rpy="0 0 0"/>
-        <mass value="0.5"/>
+        <mass value="0.477"/>
         <inertia
           ixx="0.0013" ixy="0" ixz="0"
@@ -53,5 +53,4 @@
       <xacro:insert_block name="joint_pose" />
       <axis xyz="0 1 0" />
-      <dynamics damping="0.7" friction="0.7"/>
     </joint>
     <!-- In reality, Jackal has only two motors, one per side. However, it's more
@@ -214,4 +213,19 @@
     <origin xyz="${mount_spacing} 0 0" />
   </joint>
+  <!-- <link name="gps_mount">
+    <pose>0 0 1 0 0 0</pose>
+    <sensor name="gps_sensor" type="gps">
+      <plugin name="gps_plugin" filename="libgazebo_gps_plugin.so">
+        <update_rate>10</update_rate>
+        <gpsNoise>false</gpsNoise>
+        <topic>gps/new</topic>
+      </plugin>
+    </sensor>
+  </link>
+  <joint name="gps_mount_joint" type="fixed">
+    <parent link="mid_mount" />
+    <child link="gps_mount" />
+    <origin xyz="${mount_spacing} 0 0" />
+  </joint> -->
   <!-- Bring in simulation data for Gazebo. -->
   <xacro:include filename="jackal.gazebo"/>
@@ -220,3 +234,157 @@
   <!-- Optional custom accessories. -->
   <xacro:include filename="custom_accessories.urdf.xacro" />
+<link name="front_realsense" />
+  <!--
+    The gazebo plugin aligns the depth data with the Z axis, with X=left and Y=up
+    ROS expects the depth data along the X axis, with Y=left and Z=up
+    This link only exists to give the gazebo plugin the correctly-oriented frame
+  -->
+  <link name="front_realsense_gazebo" />
+  <joint name="front_realsense_gazebo_joint" type="fixed">
+    <parent link="front_realsense"/>
+    <child link="front_realsense_gazebo"/>
+    <origin xyz="0.0 0 0" rpy="-1.5707963267948966 0 -1.5707963267948966"/>
+  </joint>
+  <gazebo reference="front_realsense">
+    <turnGravityOff>true</turnGravityOff>
+    <sensor type="depth" name="front_realsense_depth">
+      <update_rate>30</update_rate>
+      <camera>
+        <!-- 75x65 degree FOV for the depth sensor -->
+        <horizontal_fov>1.5184351666666667</horizontal_fov>
+        <vertical_fov>1.0122901111111111</vertical_fov>
+        <image>
+          <width>1280</width>
+          <height>720</height>
+          <format>R8G8B8</format>
+        </image>
+        <clip>
+          <!-- give the color sensor a maximum range of 50m so that the simulation renders nicely -->
+          <near>0.01</near>
+          <far>50.0</far>
+        </clip>
+      </camera>
+      <plugin name="kinect_controller" filename="libgazebo_ros_openni_kinect.so">
+        <baseline>0.2</baseline>
+        <alwaysOn>true</alwaysOn>
+        <updateRate>30</updateRate>
+        <cameraName>realsense</cameraName>
+        <imageTopicName>color/image_raw</imageTopicName>
+        <cameraInfoTopicName>color/camera_info</cameraInfoTopicName>
+        <depthImageTopicName>depth/image_rect_raw</depthImageTopicName>
+        <depthImageInfoTopicName>depth/camera_info</depthImageInfoTopicName>
+        <pointCloudTopicName>depth/color/points</pointCloudTopicName>
+        <frameName>$(arg namespace)/front_realsense_gazebo</frameName>
+        <pointCloudCutoff>0.105</pointCloudCutoff>
+        <pointCloudCutoffMax>8.0</pointCloudCutoffMax>
+        <!-- <distortionK1>0.00000001</distortionK1> -->
+        <!-- <distortionK2>0.00000001</distortionK2> -->
+        <!-- <distortionK3>0.00000001</distortionK3> -->
+        <!-- <distortionT1>0.00000001</distortionT1> -->
+        <!-- <distortionT2>0.00000001</distortionT2> -->
+        <CxPrime>0</CxPrime>
+        <Cx>0</Cx>
+        <Cy>0</Cy>
+        <focalLength>0</focalLength>
+        <hackBaseline>0</hackBaseline>
+      </plugin>
+    </sensor>
+  </gazebo>
+  <link name="front_realsense_lens">
+    <visual>
+      <origin xyz="0.02 0 0" rpy="${pi/2} 0 ${pi/2}" />
+      <geometry>
+        <mesh filename="package://realsense2_description/meshes/d435.dae" />
+      </geometry>
+      <material name="white" />
+    </visual>
+  </link>
+  <joint type="fixed" name="front_realsense_lens_joint">
+    <!-- Offset the camera 5cm forwards and 1cm up -->
+    <origin xyz="0.05 0 0.01" rpy="0 0 0" />
+    <parent link="front_mount" />
+    <child link="front_realsense_lens" />
+  </joint>
+  <joint type="fixed" name="front_realsense_joint">
+    <origin xyz="0.025 0 0" rpy="0 0 0" />
+    <parent link="front_realsense_lens" />
+    <child link="front_realsense" />
+  </joint>
+<link name="side_realsense" />
+  <!--
+    The gazebo plugin aligns the depth data with the Z axis, with X=left and Y=up
+    ROS expects the depth data along the X axis, with Y=left and Z=up
+    This link only exists to give the gazebo plugin the correctly-oriented frame
+  -->
+  <link name="side_realsense_gazebo" />
+  <joint name="side_realsense_gazebo_joint" type="fixed">
+    <parent link="side_realsense"/>
+    <child link="side_realsense_gazebo"/>
+    <origin xyz="0.0 0 0.05" rpy="-1.5707963267948966 0 -1.5707963267948966"/>
+  </joint>
+  <gazebo reference="side_realsense">
+    <turnGravityOff>true</turnGravityOff>
+    <sensor type="depth" name="side_realsense_depth">
+      <update_rate>30</update_rate>
+      <camera>
+        <!-- 75x65 degree FOV for the depth sensor -->
+        <horizontal_fov>1.5184351666666667</horizontal_fov>
+        <vertical_fov>1.0122901111111111</vertical_fov>
+        <image>
+          <width>1280</width>
+          <height>720</height>
+          <format>R8G8B8</format>
+        </image>
+        <clip>
+          <!-- give the color sensor a maximum range of 50m so that the simulation renders nicely -->
+          <near>0.01</near>
+          <far>50.0</far>
+        </clip>
+      </camera>
+      <plugin name="kinect_controller" filename="libgazebo_ros_openni_kinect.so">
+        <baseline>0.2</baseline>
+        <alwaysOn>true</alwaysOn>
+        <updateRate>30</updateRate>
+        <cameraName>side_realsense</cameraName>
+        <imageTopicName>color/image_raw</imageTopicName>
+        <cameraInfoTopicName>color/camera_info</cameraInfoTopicName>
+        <depthImageTopicName>depth/image_rect_raw</depthImageTopicName>
+        <depthImageInfoTopicName>depth/camera_info</depthImageInfoTopicName>
+        <pointCloudTopicName>depth/color/points</pointCloudTopicName>
+        <frameName>$(arg namespace)/side_realsense_gazebo</frameName>
+        <pointCloudCutoff>0.105</pointCloudCutoff>
+        <pointCloudCutoffMax>8.0</pointCloudCutoffMax>
+        <!-- <distortionK1>0.00000001</distortionK1> -->
+        <!-- <distortionK2>0.00000001</distortionK2> -->
+        <!-- <distortionK3>0.00000001</distortionK3> -->
+        <!-- <distortionT1>0.00000001</distortionT1> -->
+        <!-- <distortionT2>0.00000001</distortionT2> -->
+        <CxPrime>0</CxPrime>
+        <Cx>0</Cx>
+        <Cy>0</Cy>
+        <focalLength>0</focalLength>
+        <hackBaseline>0</hackBaseline>
+      </plugin>
+    </sensor>
+  </gazebo>
+  <link name="side_realsense_lens">
+    <visual>
+      <origin xyz="0.02 0 0" rpy="${pi/2} 0 -${pi/2}" />
+      <geometry>
+        <mesh filename="package://realsense2_description/meshes/d435.dae" />
+      </geometry>
+      <material name="white" />
+    </visual>
+  </link>
+  <joint type="fixed" name="side_realsense_lens_joint">
+    <!-- Offset the camera 5cm forwards and 1cm up -->
+    <origin xyz="0.05 0 0.01" rpy="0 0 0" />
+    <parent link="side_mount" />
+    <child link="side_realsense_lens" />
+  </joint>
+  <joint type="fixed" name="side_realsense_joint">
+    <origin xyz="0.025 0 0" rpy="0 0 0" />
+    <parent link="side_realsense_lens" />
+    <child link="side_realsense" />
+  </joint>
 </robot>
