Commit message: Adding changes from durable_gazebo_simulation

File: src/Multi_Robot_Simulation/urdf/evora_farm.urdf.xacro (robot description, xacro)
@@ -10,5 +10,5 @@
       <origin xyz="0 0 0" rpy="0 0 0"/>
       <geometry>
-        <mesh filename="package://durable_gazebo_simulation/meshes/evora_farm.dae"/>
+        <mesh filename="package://multi_ugv/meshes/evora_farm.dae"/>
       </geometry>
     </visual>
@@ -16,5 +16,5 @@
       <origin xyz="0 0 0" rpy="0 0 0"/>
       <geometry>
-        <mesh filename="package://durable_gazebo_simulation/meshes/evora_farm.dae"/>
+        <mesh filename="package://multi_ugv/meshes/evora_farm.dae"/>
       </geometry>
     </collision>

File: src/Multi_Robot_Simulation/urdf/solar.urdf.xacro (robot description, xacro)
@@ -10,5 +10,5 @@
       <origin xyz="0 0 0" rpy="0 0 0"/>
       <geometry>
-        <mesh filename="package://durable_gazebo_simulation/meshes/solar_farm.dae"/>
+        <mesh filename="package://multi_ugv/meshes/solar_farm.dae"/>
       </geometry>
     </visual>
@@ -16,5 +16,5 @@
       <origin xyz="0 0 0" rpy="0 0 0"/>
       <geometry>
-        <mesh filename="package://durable_gazebo_simulation/meshes/solar_farm.dae"/>
+        <mesh filename="package://multi_ugv/meshes/solar_farm.dae"/>
       </geometry>
     </collision>
